File: eagle/lipo_warner/lipo_warn.brd (EAGLE design)
At the start: 34 x 22.9 mm, 17 parts, among them IC1 ATTINY13-20SU, T1 IRLML 2244, T2 IRLML 2244

Commit message: add lable
add label for V0.1
Other:
- board size 34 x 22.9 mm -> 32.7 x 22.9 mm
- board text added: "Samuel Munz DHBW-Stuttg. V0.1"
Changed lines of the file:
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@@
 <board>
 <plain>
-<wire x1="0" y1="0" x2="33.96" y2="0" width="0" layer="20"/>
-<wire x1="33.96" y1="0" x2="33.96" y2="22.85" width="0" layer="20"/>
-<wire x1="33.96" y1="22.85" x2="0" y2="22.85" width="0" layer="20"/>
+<wire x1="0" y1="0" x2="32.69" y2="0" width="0" layer="20"/>
+<wire x1="32.69" y1="0" x2="32.69" y2="22.85" width="0" layer="20"/>
+<wire x1="32.69" y1="22.85" x2="0" y2="22.85" width="0" layer="20"/>
 <wire x1="0" y1="22.85" x2="0" y2="0" width="0" layer="20"/>
 <rectangle x1="7.62" y1="13.97" x2="10.16" y2="19.05" layer="41"/>
@@
 <wire x1="13.97" y1="15.24" x2="13.97" y2="12.7" width="1.778" layer="41"/>
 <wire x1="13.97" y1="12.7" x2="13.97" y2="11.43" width="1.778" layer="41"/>
+<text x="31.75" y="1.27" size="0.8128" layer="41" font="vector" rot="R90">Samuel Munz DHBW-Stuttg. V0.1</text>
 </plain>
 <attributes>
@@
 <contactref element="C1" pad="2"/>
 <polygon width="0.4064" layer="1" spacing="2.1844" isolate="0.254">
-<vertex x="0" y="21.59"/>
-<vertex x="33.02" y="21.59"/>
+<vertex x="0" y="22.86"/>
+<vertex x="33.02" y="22.86"/>
 <vertex x="33.02" y="0"/>
 <vertex x="0" y="0"/>
